File: hardware/utilidong-lipo-charger+septic-sepic-mk-1.0.sch (EAGLE design)
At the start: 29 parts, among them IC1 LT1610, IC2 MCP73831, Q1 N-MOSFET

Commit message: new version of lipo charger with system load balancing
Parts:
- D1: device A_butts:DIODE-SCHOTTKYMBRA140 -> A_butts:DIODE-SCHOTTKYSMA
Changed lines of the file:
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@@
 <part name="C7" library="A_butts" deviceset="CAPACITOR-CERAMIC" device="C0805" value="1uF"/>
 <part name="C8" library="A_butts" deviceset="CAPACITOR-CERAMIC" device="C0805" value="1uF"/>
-<part name="D1" library="A_butts" deviceset="DIODE-SCHOTTKY" device="MBRA140" value="MBRA140"/>
+<part name="D1" library="A_butts" deviceset="DIODE-SCHOTTKY" device="SMA" value="MBRA140"/>
 <part name="L1" library="A_butts" deviceset="INDUCTOR" device="TAIYO-YUDEN-40XX" value="22uH"/>
 <part name="L2" library="A_butts" deviceset="INDUCTOR" device="TAIYO-YUDEN-40XX" value="22uH"/>
@@
 </sheet>
 </sheets>
+<errors>
+</errors>
 </schematic>
 </drawing>

Commit message: twiddling around
Parts:
- removed C2, C4: 10uF, A_butts:CAPACITOR-CERAMICC1206
- C1, C3: value 100nF -> 4.7uF
- C5: value 22uF -> 10uF; device A_butts:CAPACITOR-POLARIZEDE2.5-6 -> A_butts:CAPACITOR-CERAMICC0805
- ZD1: device A_butts:DIODE-ZENERSOT23 -> A_butts:DIODE-ZENERSOD123
Connections:
- net 5V: no longer C2.1
- net GND: now also C5.2; no longer C2.2, C4.2, C5.-
- net VBATT+: no longer C4.1
- net VIN: now also C5.1; no longer C5.+
Changed lines of the file:
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@@
 <part name="SUPPLY3" library="A_butts" deviceset="5V" device=""/>
 <part name="GND1" library="A_butts" deviceset="GND" device=""/>
-<part name="C2" library="A_butts" deviceset="CAPACITOR-CERAMIC" device="C1206" value="10uF"/>
-<part name="C1" library="A_butts" deviceset="CAPACITOR-CERAMIC" device="C0805" value="100nF"/>
-<part name="GND6" library="A_butts" deviceset="GND" device=""/>
+<part name="C1" library="A_butts" deviceset="CAPACITOR-CERAMIC" device="C0805" value="4.7uF"/>
 <part name="SUPPLY7" library="A_butts" deviceset="5V" device=""/>
-<part name="SUPPLY8" library="A_butts" deviceset="5V" device=""/>
 <part name="SUPPLY4" library="A_butts" deviceset="5V" device=""/>
 <part name="GND8" library="A_butts" deviceset="GND" device=""/>
@@
 <part name="R5" library="A_butts" deviceset="RESISTOR" device="R0805" value="10k"/>
 <part name="U$3" library="A_butts" deviceset="VBATT+" device=""/>
-<part name="C4" library="A_butts" deviceset="CAPACITOR-CERAMIC" device="C1206" value="10uF"/>
-<part name="GND11" library="A_butts" deviceset="GND" device=""/>
-<part name="U$4" library="A_butts" deviceset="VBATT+" device=""/>
 <part name="OUT" library="A_butts" deviceset="M02" device="PTH-CENTERED-R+"/>
-<part name="C3" library="A_butts" deviceset="CAPACITOR-CERAMIC" device="C0805" value="100nF"/>
+<part name="C3" library="A_butts" deviceset="CAPACITOR-CERAMIC" device="C0805" value="4.7uF"/>
 <part name="U$6" library="A_butts" deviceset="VBATT+" device=""/>
 <part name="GND2" library="A_butts" deviceset="GND" device=""/>
@@
 <part name="R1" library="A_butts" deviceset="RESISTOR" device="R0805" value="1M"/>
 <part name="R2" library="A_butts" deviceset="RESISTOR" device="R0805" value="604k"/>
-<part name="C5" library="A_butts" deviceset="CAPACITOR-POLARIZED" device="E2.5-6" value="22uF"/>
 <part name="C6" library="A_butts" deviceset="CAPACITOR-POLARIZED" device="E2.5-6" value="22uF"/>
 <part name="C7" library="A_butts" deviceset="CAPACITOR-CERAMIC" device="C0805" value="1uF"/>
@@
 <part name="U$10" library="A_butts" deviceset="VBATT+" device=""/>
 <part name="D2" library="A_butts" deviceset="DIODE-SCHOTTKY" device="MBRA140" value="MBRA140"/>
-<part name="ZD1" library="A_butts" deviceset="DIODE-ZENER" device="SOT23" value="10V"/>
+<part name="ZD1" library="A_butts" deviceset="DIODE-ZENER" device="SOD123" value="10V"/>
 <part name="SUPPLY6" library="A_butts" deviceset="5V" device=""/>
 <part name="SUPPLY9" library="A_butts" deviceset="VIN" device=""/>
 <part name="D3" library="A_butts" deviceset="DIODE-SCHOTTKY" device="MBRA140" value="MBRA140"/>
+<part name="C5" library="A_butts" deviceset="CAPACITOR-CERAMIC" device="C0805" value="10uF"/>
 </parts>
 <sheets>
@@
 <instance part="SUPPLY3" gate="G$1" x="66.04" y="165.1"/>
 <instance part="GND1" gate="1" x="45.72" y="111.76"/>
-<instance part="C2" gate="G$1" x="58.42" y="121.92"/>
 <instance part="C1" gate="G$1" x="45.72" y="121.92"/>
-<instance part="GND6" gate="1" x="58.42" y="111.76"/>
 <instance part="SUPPLY7" gate="G$1" x="45.72" y="129.54"/>
-<instance part="SUPPLY8" gate="G$1" x="58.42" y="129.54"/>
 <instance part="SUPPLY4" gate="G$1" x="101.6" y="137.16"/>
 <instance part="GND8" gate="1" x="127" y="114.3"/>
@@
 <instance part="R5" gate="G$1" x="182.88" y="172.72"/>
 <instance part="U$3" gate="1" x="167.64" y="137.16"/>
-<instance part="C4" gate="G$1" x="83.82" y="121.92"/>
-<instance part="GND11" gate="1" x="83.82" y="111.76"/>
-<instance part="U$4" gate="1" x="83.82" y="129.54"/>
 <instance part="OUT" gate="G$1" x="215.9" y="134.62" rot="MR0"/>
 <instance part="C3" gate="G$1" x="71.12" y="121.92"/>
@@
 <instance part="R1" gate="G$1" x="175.26" y="86.36" rot="MR270"/>
 <instance part="R2" gate="G$1" x="175.26" y="71.12" rot="MR270"/>
-<instance part="C5" gate="G$1" x="93.98" y="73.66" rot="MR0"/>
 <instance part="C6" gate="G$1" x="185.42" y="78.74" rot="MR0"/>
 <instance part="C7" gate="G$1" x="154.94" y="93.98" rot="MR90"/>
@@
 <instance part="SUPPLY9" gate="G$1" x="68.58" y="66.04"/>
 <instance part="D3" gate="G$1" x="60.96" y="53.34"/>
+<instance part="C5" gate="G$1" x="93.98" y="73.66" rot="MR0"/>
 </instances>
 <busses>
@@
 <pinref part="C1" gate="G$1" pin="2"/>
 <wire x1="45.72" y1="116.84" x2="45.72" y2="114.3" width="0.1524" layer="91"/>
-</segment>
-<segment>
-<pinref part="C2" gate="G$1" pin="2"/>
-<pinref part="GND6" gate="1" pin="GND"/>
-<wire x1="58.42" y1="116.84" x2="58.42" y2="114.3" width="0.1524" layer="91"/>
 </segment>
 <segment>
@@
 </segment>
 <segment>
-<pinref part="C4" gate="G$1" pin="2"/>
-<pinref part="GND11" gate="1" pin="GND"/>
-<wire x1="83.82" y1="116.84" x2="83.82" y2="114.3" width="0.1524" layer="91"/>
-</segment>
-<segment>
 <pinref part="USB1" gate="G$1" pin="GND"/>
 <wire x1="63.5" y1="152.4" x2="66.04" y2="152.4" width="0.1524" layer="91"/>
@@
 </segment>
 <segment>
-<pinref part="C5" gate="G$1" pin="-"/>
 <wire x1="93.98" y1="50.8" x2="93.98" y2="53.34" width="0.1524" layer="91"/>
 <pinref part="GND7" gate="1" pin="GND"/>
@@
 <wire x1="203.2" y1="50.8" x2="203.2" y2="53.34" width="0.1524" layer="91"/>
 <junction x="203.2" y="53.34"/>
+<pinref part="C5" gate="G$1" pin="2"/>
 </segment>
 </net>
@@
 <pinref part="SUPPLY7" gate="G$1" pin="5V"/>
 <wire x1="45.72" y1="129.54" x2="45.72" y2="127" width="0.1524" layer="91"/>
-</segment>
-<segment>
-<pinref part="C2" gate="G$1" pin="1"/>
-<pinref part="SUPPLY8" gate="G$1" pin="5V"/>
-<wire x1="58.42" y1="129.54" x2="58.42" y2="127" width="0.1524" layer="91"/>
 </segment>
 <segment>
@@
 </segment>
 <segment>
-<pinref part="U$4" gate="1" pin="VBATT+"/>
-<pinref part="C4" gate="G$1" pin="1"/>
-<wire x1="83.82" y1="129.54" x2="83.82" y2="127" width="0.1524" layer="91"/>
-</segment>
-<segment>
 <pinref part="IC2" gate="A" pin="VBAT"/>
 <wire x1="165.1" y1="134.62" x2="167.64" y2="134.62" width="0.1524" layer="91"/>
@@
 <net name="VIN" class="0">
 <segment>
-<pinref part="C5" gate="G$1" pin="+"/>
 <wire x1="93.98" y1="78.74" x2="93.98" y2="93.98" width="0.1524" layer="91"/>
 <wire x1="93.98" y1="93.98" x2="116.84" y2="93.98" width="0.1524" layer="91"/>
@@
 <pinref part="SUPPLY1" gate="G$1" pin="VIN"/>
 <wire x1="93.98" y1="93.98" x2="93.98" y2="96.52" width="0.1524" layer="91"/>
-</segment>
-<segment>
+<pinref part="C5" gate="G$1" pin="1"/>
+</segment>
+<segment>
