File: hardware/utilidong-ftdi-uart-mk-2.2.sch (EAGLE design)
At the start: 13 parts, among them U1 FTS31XS

Commit message: almost finished way smaller form factor, now flipped to the correct orientation
Parts:
- C2, C3: device a_parts:CAPACITOR-CERAMICC0603 -> a_parts:CAPACITOR-CERAMICC0603-TIGHTER
- R6, R7: device a_parts:RESISTORR0603 -> a_parts:RESISTORR0603-TIGHTER
- RX, TX: value LED0603 -> LED0603-TIGHT; device a_parts:LED0603 -> a_parts:LED0603-TIGHT
- U2: value (none) -> V_REG_SOT-23-5SPX3819; device a_parts:VREG_1117SOT89 -> a_parts:V_REG_SOT-23-5SPX3819
- UART: value FTDI_3V3 -> FTDI_CONNSMT_FEMALE_RA_3V3_FLIPPED; device a_parts:FTDI_3V3 -> a_parts:FTDI_CONNSMT_FEMALE_RA_3V3_FLIPPED
- USB: value (none) -> USB-AB-SHIELDFCI-10103594-USB-MICRO-B-EVENLESS; device a_parts:USB-ABFCI-10103594-USB-MICRO-B-LESS -> a_parts:USB-AB-SHIELDFCI-10103594-USB-MICRO-B-EVENLESS
Connections:
- net 3.3V: now also U2.OUT, UART.VCC; no longer U2.VOUT, UART.3V3
- net 5V: now also U2.EN, U2.IN; no longer U2.VIN
Other:
- moved on the sheet: C1, C2, C4
